File: Hackpad/Hackpad.kicad_sch (KiCad schematic)
At the start: 8 parts, among them SW1 SW_Push, SW2 SW_Push, SW3 SW_Push, SW4 SW_Push, SW5 RotaryEncoder, U1 XIAO-RP2040-DIP

Commit message: updated pcb
Parts:
- added SW10, SW6, SW7, SW8, SW9: SW_Push, Button_Switch_Keyboard:SW_Cherry_MX_1.00u_PCB, symbol Switch:SW_Push
Connections:
- net GND: now also SW10.2, SW6.2, SW7.2, SW8.2, SW9.2
- net at U1.2 (GPIO27/ADC1/A1): now also SW10.1
- net at U1.3 (GPIO28/ADC2/A2): now also SW6.1
- net at U1.4 (GPIO29/ADC3/A3): now also SW7.1
- net at U1.6 (GPIO7/SCL): now also SW8.1
- net at U1.7 (GPIO0/TX): now also SW9.1

Commit message: finished pcb
Parts:
- removed SW5: RotaryEncoder, Rotary_Encoder:RotaryEncoder_Alps_EC11E-Switch_Vertical_H20mm, symbol Device:RotaryEncoder
Changed lines of the file:
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@@
-	)
-	(symbol
-		(lib_id "Device:RotaryEncoder")
-		(at 138.43 64.77 0)
-		(unit 1)
-		(exclude_from_sim no)
-		(in_bom yes)
-		(on_board yes)
-		(dnp no)
-		(fields_autoplaced yes)
-		(property "Reference" "SW5"
-			(at 144.78 63.4999 0)
-			(effects
-				(font
-					(size 1.27 1.27)
-				)
-				(justify left)
-			)
-		)
-		(property "Value" "RotaryEncoder"
-			(at 144.78 66.0399 0)
-			(effects
-				(font
-					(size 1.27 1.27)
-				)
-				(justify left)
-			)
-		)
-		(property "Footprint" "Rotary_Encoder:RotaryEncoder_Alps_EC11E-Switch_Vertical_H20mm"
-			(at 134.62 60.706 0)
-			(effects
-				(font
-					(size 1.27 1.27)
-				)
-				(hide yes)
-			)
-		)
-		(property "Datasheet" "~"
-			(at 138.43 58.166 0)
-			(effects
-				(font
-					(size 1.27 1.27)
-				)
-				(hide yes)
-			)
-		)
-		(property "Description" "Rotary encoder, dual channel, incremental quadrate outputs"
-			(at 138.43 64.77 0)
-			(effects
-				(font
-					(size 1.27 1.27)
-				)
-				(hide yes)
-			)
-		)
-		(pin "B"
-		)
-		(pin "C"
-		)
-		(pin "A"
-		)
-		(instances
-			(project "Hackpad"
-				(path "/cbc0698d-34bf-490d-b65b-ac0022947fdb"
-					(reference "SW5")
-					(unit 1)
-				)
-			)
-		)
 	)
 	(symbol
